File: module/hw/sch_pcb/module.kicad_pcb (KiCad board)
At the start: 2 copper layers, 0 parts

Commit message: template update
Other:
- net class MLAB_default added: clearance 0.2, trace_width 0.45, via_dia 0.6, via_drill 0.4
- net class MLAB_power added: clearance 0.4, trace_width 0.7, via_dia 0.8, via_drill 0.6
Changed lines of the file:
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@@
-(kicad_pcb (version 4) (host pcbnew "(2015-04-05 BZR 5577)-product")
+(kicad_pcb (version 20171130) (host pcbnew 5.0.0-rc2-dev-unknown-5f578c8~62~ubuntu16.04.1)
   (general
-    (links 0)
-    (no_connects 0)
-    (area 0 0 0 0)
     (thickness 1.6)
     (drawings 0)
@@
     (0 F.Cu signal)
     (31 B.Cu signal)
-    (32 B.Adhes user)
-    (33 F.Adhes user)
     (34 B.Paste user)
-    (35 F.Paste user)
     (36 B.SilkS user)
     (37 F.SilkS user)
     (38 B.Mask user)
     (39 F.Mask user)
-    (40 Dwgs.User user)
-    (41 Cmts.User user)
-    (42 Eco1.User user)
-    (43 Eco2.User user)
     (44 Edge.Cuts user)
-    (45 Margin user)
-    (46 B.CrtYd user)
-    (47 F.CrtYd user)
-    (48 B.Fab user)
-    (49 F.Fab user)
   )
   (setup
@@
       (layerselection 0x00030_80000001)
       (usegerberextensions false)
+      (usegerberattributes false)
+      (usegerberadvancedattributes false)
+      (creategerberjobfile false)
       (excludeedgelayer true)
       (linewidth 0.150000)
@@
       (hpglpenspeed 20)
       (hpglpendiameter 15)
-      (hpglpenoverlay 2)
       (psnegative false)
       (psa4output false)
@@
     (uvia_dia 0.3)
     (uvia_drill 0.1)
+  )
+  (net_class MLAB_default ""
+    (clearance 0.2)
+    (trace_width 0.45)
+    (via_dia 0.6)
+    (via_drill 0.4)
+    (uvia_dia 0.3)
+    (uvia_drill 0.1)
+  )
+  (net_class MLAB_power ""
+    (clearance 0.4)
+    (trace_width 0.7)
+    (via_dia 0.8)
+    (via_drill 0.6)
+    (uvia_dia 0.3)
+    (uvia_drill 0.1)

Commit message: KiCAD template edited
Other:
- net class Default: trace_width 0.25 -> 0.5; via_dia 0.6 -> 0.8
- net class MLAB_default removed
- rule trace_min: 0.2 -> 0.4
Changed lines of the file:
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@@
-(kicad_pcb (version 20171130) (host pcbnew 5.0.0-rc2-dev-unknown-5f578c8~62~ubuntu16.04.1)
+(kicad_pcb (version 20171130) (host pcbnew 6.0.0-rc1-unknown-1a22918~65~ubuntu18.04.1)
   (general
     (thickness 1.6)
@@
     (39 F.Mask user)
     (44 Edge.Cuts user)
+    (45 Margin user)
+    (46 B.CrtYd user)
+    (47 F.CrtYd user)
+    (48 B.Fab user)
+    (49 F.Fab user)
   )
   (setup
-    (last_trace_width 0.25)
+    (last_trace_width 0.5)
     (trace_clearance 0.2)
     (zone_clearance 0.508)
     (zone_45_only no)
-    (trace_min 0.2)
+    (trace_min 0.4)
     (segment_width 0.2)
     (edge_width 0.15)
-    (via_size 0.6)
+    (via_size 0.8)
     (via_drill 0.4)
     (via_min_size 0.4)
     (via_min_drill 0.3)
-    (uvia_size 0.3)
-    (uvia_drill 0.1)
+    (uvia_size 0.4)
+    (uvia_drill 0.2)
     (uvias_allowed no)
     (uvia_min_size 0.2)
@@
     (pad_to_mask_clearance 0.2)
     (aux_axis_origin 0 0)
-    (visible_elements FFFFFF7F)
+    (visible_elements FFFFEF7F)
     (pcbplotparams
       (layerselection 0x00030_80000001)
@@
       (hpglpennumber 1)
       (hpglpenspeed 20)
-      (hpglpendiameter 15)
+      (hpglpendiameter 15.000000)
       (psnegative false)
       (psa4output false)
@@
   (net_class Default "This is the default net class."
     (clearance 0.2)
-    (trace_width 0.25)
-    (via_dia 0.6)
+    (trace_width 0.5)
+    (via_dia 0.8)
     (via_drill 0.4)
-    (uvia_dia 0.3)
-    (uvia_drill 0.1)
-  )
-  (net_class MLAB_default ""
-    (clearance 0.2)
-    (trace_width 0.45)
-    (via_dia 0.6)
-    (via_drill 0.4)
-    (uvia_dia 0.3)
-    (uvia_drill 0.1)
+    (uvia_dia 0.4)
+    (uvia_drill 0.2)
+    (diff_pair_gap 0.25)
+    (diff_pair_width 0.4)
   )
   (net_class MLAB_power ""
@@
     (via_dia 0.8)
     (via_drill 0.6)
-    (uvia_dia 0.3)
-    (uvia_drill 0.1)
+    (uvia_dia 0.4)
+    (uvia_drill 0.2)
+    (diff_pair_gap 0.25)
+    (diff_pair_width 0.4)
   )
 )
