File: module/hw/sch_pcb/module.sch (KiCad schematic (older format))
At the start: 8 parts, among them J1 Umin ... Umax, M1 HOLE, M2 HOLE, M3 HOLE, M4 HOLE

Commit message: template update
Parts:
- C1: symbol CP_Small -> Device:CP_Small
- C2: symbol C_Small -> Device:C_Small
- D1: symbol D_Small -> Device:D_Small
- J1: value Umin ... Umax -> 0 ... Umax; symbol HEADER_2x03_PARALLEL -> MLAB_HEADER:HEADER_2x03_PARALLEL
- M1, M2, M3, M4: symbol HOLE -> MLAB_MECHANICAL:HOLE
Changed lines of the file:
@@
-EESchema Schematic File Version 2
-LIBS:74xgxx
-LIBS:74xx
-LIBS:ac-dc
-LIBS:actel
-LIBS:adc-dac
-LIBS:Altera
-LIBS:analog_devices
-LIBS:analog_switches
-LIBS:atmel
-LIBS:audio
-LIBS:brooktre
-LIBS:cmos4000
-LIBS:cmos_ieee
-LIBS:conn
-LIBS:contrib
-LIBS:cypress
-LIBS:dc-dc
-LIBS:device
-LIBS:digital-audio
-LIBS:diode
-LIBS:display
-LIBS:dsp
-LIBS:elec-unifil
-LIBS:ESD_Protection
-LIBS:ftdi
-LIBS:gennum
-LIBS:graphic
-LIBS:hc11
-LIBS:intel
-LIBS:interface
-LIBS:ir
-LIBS:Lattice
-LIBS:linear
-LIBS:logo
-LIBS:maxim
-LIBS:memory
-LIBS:microchip_dspic33dsc
-LIBS:microchip
-LIBS:microchip_pic10mcu
-LIBS:microchip_pic12mcu
-LIBS:microchip_pic16mcu
-LIBS:microchip_pic18mcu
-LIBS:microchip_pic32mcu
-LIBS:microcontrollers
-LIBS:motor_drivers
-LIBS:motorola
-LIBS:msp430
-LIBS:nordicsemi
-LIBS:nxp_armmcu
-LIBS:onsemi
-LIBS:opto
-LIBS:Oscillators
-LIBS:philips
-LIBS:powerint
-LIBS:power
-LIBS:Power_Management
-LIBS:pspice
-LIBS:references
-LIBS:regul
-LIBS:relays
-LIBS:rfcom
-LIBS:sensors
-LIBS:silabs
-LIBS:siliconi
-LIBS:stm32
-LIBS:stm8
-LIBS:supertex
-LIBS:switches
-LIBS:texas
-LIBS:transf
-LIBS:transistors
-LIBS:ttl_ieee
-LIBS:valves
-LIBS:video
-LIBS:Xicor
-LIBS:xilinx
-LIBS:Zilog
-LIBS:module-cache
-EELAYER 25 0
+EESchema Schematic File Version 4
+EELAYER 26 0
 EELAYER END
 $Descr A4 11693 8268
@@
 $EndDescr
 $Comp
-L HEADER_2x03_PARALLEL J1
+L MLAB_HEADER:HEADER_2x03_PARALLEL J1
 U 1 1 549D65BC
 P 10550 1050
 F 0 "J1" H 10550 850 60  0000 C CNN
-F 1 "Umin ... Umax" H 10550 1250 60  0000 C CNN
+F 1 "0 ... Umax" H 10550 1250 60  0000 C CNN
 F 2 "" H 10550 1150 60  0000 C CNN
 F 3 "" H 10550 1150 60  0000 C CNN
@@
 $EndComp
 $Comp
-L VCC #PWR1
+L power:VCC #PWR1
 U 1 1 549D7353
 P 9350 1000
@@
 $EndComp
 $Comp
-L GND #PWR2
+L power:GND #PWR2
 U 1 1 549D73B2
 P 9350 1400
@@
 POWER INPUT
 $Comp
-L HOLE M1
+L MLAB_MECHANICAL:HOLE M1
 U 1 1 549D7549
 P 10050 1900
@@
 $EndComp
 $Comp
-L HOLE M2
+L MLAB_MECHANICAL:HOLE M2
 U 1 1 549D7628
 P 10250 1900
@@
 $EndComp
 $Comp
-L HOLE M3
+L MLAB_MECHANICAL:HOLE M3
 U 1 1 549D7646
 P 10450 1900
@@
 $EndComp
 $Comp
-L HOLE M4
+L MLAB_MECHANICAL:HOLE M4
 U 1 1 549D7665
 P 10650 1900
@@
 $EndComp
 $Comp
-L GND #PWR3
+L power:GND #PWR3
 U 1 1 549D770F
 P 10850 1850
@@
 	10850 1850 10850 1800
 Wire Wire Line
-	10850 1800 10050 1800
+	10850 1800 10650 1800
 Wire Wire Line
 	10050 1800 10050 1850
@@
 MOUNTING HOLES
 $Comp
-L D_Small D1
+L Device:D_Small D1
 U 1 1 55622FB7
 P 9950 1200
@@
 $EndComp
 $Comp
-L C_Small C2
+L Device:C_Small C2
 U 1 1 5562302C
 P 9650 1200
@@
 $EndComp
 $Comp
-L CP_Small C1
+L Device:CP_Small C1
 U 1 1 55623093
 P 9350 1200
@@
 $EndComp
 Wire Wire Line
-	10300 1050 9350 1050
-Wire Wire Line
-	9350 1000 9350 1100
+	10300 1050 9950 1050
+Wire Wire Line
+	9350 1000 9350 1050
 Connection ~ 9350 1050
 Wire Wire Line
@@
 	10300 950  10250 950
 Wire Wire Line
-	10250 950  10250 1350
-Wire Wire Line
-	10250 1350 9350 1350
-Wire Wire Line
-	9350 1300 9350 1400
+	10250 950  10250 1150
+Wire Wire Line
+	10250 1350 9950 1350
+Wire Wire Line
+	9350 1300 9350 1350
 Connection ~ 9350 1350
 Wire Wire Line
@@
 Wire Notes Line
 	9200 750  10950 750
+Wire Wire Line
+	10250 1800 10050 1800
+Wire Wire Line
+	10450 1800 10250 1800
+Wire Wire Line
+	10650 1800 10450 1800
+Wire Wire Line
+	9350 1050 9350 1100
+Wire Wire Line
+	9650 1050 9350 1050
+Wire Wire Line
+	9950 1050 9650 1050
+Wire Wire Line
+	9350 1350 9350 1400
+Wire Wire Line
+	9650 1350 9350 1350
+Wire Wire Line
+	9950 1350 9650 1350
+Wire Wire Line
+	10250 1150 10250 1350
 $EndSCHEMATC

Commit message: KiCAD template edited
Parts:
- removed D1: M4, symbol Device:D_Small
- removed J1: 0 ... Umax, symbol MLAB_HEADER:HEADER_2x03_PARALLEL
- added D1: 0.0V, Mlab_D:Diode-MiniMELF_Standard, symbol MLAB_D:D_ZENER
- added J1: JUMP_3X2, Mlab_Pin_Headers:Straight_2x03, symbol MLAB_Jumpers:JUMP_3X2
- C1: value C/U -> 10uF; footprint (none) -> Mlab_R:SMD-0805
- C2: footprint (none) -> Mlab_R:SMD-0805; UST_id (none) -> C0805_100n
- M1, M2, M3, M4: footprint (none) -> Mlab_Mechanical:MountingHole_3mm
Connections:
- wire segments 27 -> 25
Other:
- moved on the sheet: C1, C2
Changed lines of the file:
@@
 EESchema Schematic File Version 4
+LIBS:module-cache
 EELAYER 26 0
 EELAYER END
@@
 $EndDescr
 $Comp
-L MLAB_HEADER:HEADER_2x03_PARALLEL J1
-U 1 1 549D65BC
-P 10550 1050
-F 0 "J1" H 10550 850 60  0000 C CNN
-F 1 "0 ... Umax" H 10550 1250 60  0000 C CNN
-F 2 "" H 10550 1150 60  0000 C CNN
-F 3 "" H 10550 1150 60  0000 C CNN
-	1    10550 1050
-	1    0    0    -1
-$EndComp
-$Comp
-L power:VCC #PWR1
+L power:VCC #PWR01
 U 1 1 549D7353
-P 9350 1000
-F 0 "#PWR1" H 9350 850 60  0001 C CNN
-F 1 "VCC" H 9350 1150 60  0000 C CNN
-F 2 "" H 9350 1000 60  0000 C CNN
-F 3 "" H 9350 1000 60  0000 C CNN
-	1    9350 1000
-	1    0    0    -1
-$EndComp
-$Comp
-L power:GND #PWR2
+P 9550 900
+F 0 "#PWR01" H 9550 750 60  0001 C CNN
+F 1 "VCC" H 9550 1050 60  0000 C CNN
+F 2 "" H 9550 900 60  0000 C CNN
+F 3 "" H 9550 900 60  0000 C CNN
+	1    9550 900
+	1    0    0    -1
+$EndComp
+$Comp
+L power:GND #PWR02
 U 1 1 549D73B2
-P 9350 1400
-F 0 "#PWR2" H 9350 1150 60  0001 C CNN
-F 1 "GND" H 9350 1250 60  0000 C CNN
-F 2 "" H 9350 1400 60  0000 C CNN
-F 3 "" H 9350 1400 60  0000 C CNN
-	1    9350 1400
-	1    0    0    -1
-$EndComp
-Text Notes 9200 1700 0    60   ~ 0
+P 9550 1400
+F 0 "#PWR02" H 9550 1150 60  0001 C CNN
+F 1 "GND" H 9550 1250 60  0000 C CNN
+F 2 "" H 9550 1400 60  0000 C CNN
+F 3 "" H 9550 1400 60  0000 C CNN
+	1    9550 1400
+	1    0    0    -1
+$EndComp
+Text Notes 9400 1700 0    60   ~ 0
 POWER INPUT
 $Comp
@@
 F 0 "M1" V 9950 1900 60  0000 C CNN
 F 1 "HOLE" H 10050 1800 60  0001 C CNN
-F 2 "" H 10050 1900 60  0000 C CNN
+F 2 "Mlab_Mechanical:MountingHole_3mm" H 10050 1900 60  0001 C CNN
 F 3 "" H 10050 1900 60  0000 C CNN
 	1    10050 1900
@@
 F 0 "M2" V 10150 1900 60  0000 C CNN
 F 1 "HOLE" H 10250 1800 60  0001 C CNN
-F 2 "" H 10250 1900 60  0000 C CNN
+F 2 "Mlab_Mechanical:MountingHole_3mm" H 10250 1900 60  0001 C CNN
 F 3 "" H 10250 1900 60  0000 C CNN
 	1    10250 1900
@@
 F 0 "M3" V 10350 1900 60  0000 C CNN
 F 1 "HOLE" H 10450 1800 60  0001 C CNN
-F 2 "" H 10450 1900 60  0000 C CNN
+F 2 "Mlab_Mechanical:MountingHole_3mm" H 10450 1900 60  0001 C CNN
 F 3 "" H 10450 1900 60  0000 C CNN
 	1    10450 1900
@@
 F 0 "M4" V 10550 1900 60  0000 C CNN
 F 1 "HOLE" H 10650 1800 60  0001 C CNN
-F 2 "" H 10650 1900 60  0000 C CNN
+F 2 "Mlab_Mechanical:MountingHole_3mm" H 10650 1900 60  0001 C CNN
 F 3 "" H 10650 1900 60  0000 C CNN
 	1    10650 1900
@@
 $EndComp
 $Comp
-L power:GND #PWR3
+L power:GND #PWR03
 U 1 1 549D770F
 P 10850 1850
-F 0 "#PWR3" H 10850 1600 60  0001 C CNN
+F 0 "#PWR03" H 10850 1600 60  0001 C CNN
 F 1 "GND" H 10850 1700 60  0000 C CNN
 F 2 "" H 10850 1850 60  0000 C CNN
@@
 MOUNTING HOLES
 $Comp
-L Device:D_Small D1
-U 1 1 55622FB7
-P 9950 1200
-F 0 "D1" V 9850 1200 50  0000 R CNN
-F 1 "M4" V 10050 1150 50  0000 R CNN
-F 2 "" V 9950 1200 60  0000 C CNN
-F 3 "" V 9950 1200 60  0000 C CNN
-	1    9950 1200
-	0    -1   1    0
-$EndComp
+L Device:CP_Small C1
+U 1 1 55623093
+P 9550 1150
+F 0 "C1" H 9550 1250 50  0000 L CNN
+F 1 "10uF" H 9550 1050 50  0000 L CNN
+F 2 "Mlab_R:SMD-0805" H 9550 1150 60  0001 C CNN
+F 3 "" H 9550 1150 60  0000 C CNN
+	1    9550 1150
+	1    0    0    -1
+$EndComp
+Connection ~ 9550 1350
+Wire Wire Line
+	10250 1800 10050 1800
+Wire Wire Line
+	10450 1800 10250 1800
+Wire Wire Line
+	10650 1800 10450 1800
+Wire Wire Line
+	9550 1350 9550 1400
+$Comp
+L MLAB_D:D_ZENER D1
+U 1 1 5B4DE0B5
+P 10150 1150
+F 0 "D1" V 10050 1150 50  0000 L CNN
+F 1 "0.0V" V 10250 1150 50  0000 L CNN
+F 2 "Mlab_D:Diode-MiniMELF_Standard" H 10150 1150 60  0001 C CNN
+F 3 "" H 10150 1150 60  0000 C CNN
+	1    10150 1150
+	0    1    1    0
+$EndComp
+Wire Wire Line
+	9550 900  9550 950
+Wire Wire Line
+	10150 950  9850 950
+Connection ~ 9550 950
+Wire Wire Line
+	9550 950  9550 1050
+Wire Wire Line
+	9550 1250 9550 1350
+$Comp
+L MLAB_Jumpers:JUMP_3X2 J1
+U 1 1 5B4DDE60
+P 10900 1000
+F 0 "J1" H 10829 1030 50  0000 L CNN
+F 1 "JUMP_3X2" V 10900 1050 40  0001 C CNN
+F 2 "Mlab_Pin_Headers:Straight_2x03" H 10900 1000 60  0001 C CNN
+F 3 "" H 10900 1000 60  0000 C CNN
+	1    10900 1000
+	1    0    0    -1
+$EndComp
+Wire Wire Line
+	10500 850  10450 850
+Wire Wire Line
+	10450 850  10450 1050
+Wire Wire Line
+	10500 1050 10450 1050
+Connection ~ 10450 1050
+Wire Wire Line
+	10450 1050 10450 1350
+Wire Notes Line
+	10950 1700 9350 1700
+Wire Notes Line
+	9350 1700 9350 700
+Wire Notes Line
+	9350 700  10950 700
+Wire Notes Line
+	10950 700  10950 1700
+Wire Wire Line
+	9850 950  9550 950
+Connection ~ 9850 950
+Wire Wire Line
+	9850 950  9850 1050
+Wire Wire Line
+	9850 1350 10150 1350
+Wire Wire Line
+	9850 1350 9550 1350
+Connection ~ 9850 1350
+Wire Wire Line
+	9850 1250 9850 1350
 $Comp
 L Device:C_Small C2
 U 1 1 5562302C
-P 9650 1200
-F 0 "C2" H 9650 1300 50  0000 L CNN
-F 1 "100nF" H 9650 1100 50  0000 L CNN
-F 2 "" H 9650 1200 60  0000 C CNN
-F 3 "" H 9650 1200 60  0000 C CNN
-	1    9650 1200
-	1    0    0    -1
-$EndComp
-$Comp
-L Device:CP_Small C1
-U 1 1 55623093
-P 9350 1200
-F 0 "C1" H 9350 1300 50  0000 L CNN
-F 1 "C/U" H 9350 1100 50  0000 L CNN
-F 2 "" H 9350 1200 60  0000 C CNN
-F 3 "" H 9350 1200 60  0000 C CNN
-	1    9350 1200
-	1    0    0    -1
-$EndComp
-Wire Wire Line
-	10300 1050 9950 1050
-Wire Wire Line
-	9350 1000 9350 1050
-Connection ~ 9350 1050
-Wire Wire Line
-	9650 1100 9650 1050
-Connection ~ 9650 1050
-Wire Wire Line
-	9950 1100 9950 1050
-Connection ~ 9950 1050
-Wire Wire Line
-	10300 950  10250 950
-Wire Wire Line
-	10250 950  10250 1150
-Wire Wire Line
-	10250 1350 9950 1350
-Wire Wire Line
-	9350 1300 9350 1350
-Connection ~ 9350 1350
-Wire Wire Line
-	9650 1300 9650 1350
-Connection ~ 9650 1350
-Wire Wire Line
-	9950 1300 9950 1350
-Connection ~ 9950 1350
-Wire Wire Line
-	10300 1150 10250 1150
-Connection ~ 10250 1150
-Wire Notes Line
-	10950 750  10950 1700
-Wire Notes Line
-	10950 1700 9200 1700
-Wire Notes Line
-	9200 1700 9200 750
-Wire Notes Line
-	9200 750  10950 750
-Wire Wire Line
-	10250 1800 10050 1800
-Wire Wire Line
-	10450 1800 10250 1800
-Wire Wire Line
-	10650 1800 10450 1800
-Wire Wire Line
-	9350 1050 9350 1100
-Wire Wire Line
-	9650 1050 9350 1050
-Wire Wire Line
-	9950 1050 9650 1050
-Wire Wire Line
-	9350 1350 9350 1400
-Wire Wire Line
-	9650 1350 9350 1350
-Wire Wire Line
-	9950 1350 9650 1350
-Wire Wire Line
-	10250 1150 10250 1350
+P 9850 1150
+F 0 "C2" H 9850 1250 50  0000 L CNN
+F 1 "100nF" H 9850 1050 50  0000 L CNN
+F 2 "Mlab_R:SMD-0805" H 9850 1150 60  0001 C CNN
+F 3 "" H 9850 1150 60  0000 C CNN
+F 4 "C0805_100n" H 9850 1150 50  0001 C CNN "UST_id"
+	1    9850 1150
+	1    0    0    -1
+$EndComp
+Connection ~ 10150 950
+Connection ~ 10150 1350
+Wire Wire Line
+	10150 1350 10450 1350
+Wire Wire Line
+	10150 950  10500 950
 $EndSCHEMATC
